Commit message: Fix bad xacro file for xv11_lidar

File: turtlebot2_description/urdf/xv11_lidar.urdf.xacro (robot description, xacro)
@@ -1,10 +1,9 @@
 <?xml version="1.0"?>
 <!-- Xacro file for XV11 LIDAR -->
-<xacro:macro name="xv11_lidar" params="parent_link">
+<xacro:macro name="xv11_lidar" parent_link="">
   <!-- XV11 LIDAR link -->
   <link name="laser_frame">
     <visual>
       <geometry>
-        <!-- Use a cylinder to represent the LIDAR -->
         <cylinder radius="0.035" length="0.02"/>
       </geometry>
@@ -12,5 +11,4 @@
         <color rgba="0.5 0.5 0.5 1.0"/>
       </material>
-      <origin xyz="0 0 0" rpy="0 0 0"/>
     </visual>
     <collision>
@@ -18,9 +16,7 @@
         <cylinder radius="0.035" length="0.02"/>
       </geometry>
-      <origin xyz="0 0 0" rpy="0 0 0"/>
     </collision>
     <inertial>
       <mass value="0.2"/>
-      <origin xyz="0 0 0" rpy="0 0 0"/>
       <inertia
         ixx="0.0001" ixy="0.0" ixz="0.0"

Commit message: Fix bad xacro file for xv11_lidar, take 2

File: turtlebot2_description/urdf/xv11_lidar.urdf.xacro (robot description, xacro)
@@ -1,33 +1,36 @@
 <?xml version="1.0"?>
-<!-- Xacro file for XV11 LIDAR -->
-<xacro:macro name="xv11_lidar" parent_link="">
-  <!-- XV11 LIDAR link -->
-  <link name="laser_frame">
-    <visual>
-      <geometry>
-        <cylinder radius="0.035" length="0.02"/>
-      </geometry>
-      <material name="grey">
-        <color rgba="0.5 0.5 0.5 1.0"/>
-      </material>
-    </visual>
-    <collision>
-      <geometry>
-        <cylinder radius="0.035" length="0.02"/>
-      </geometry>
-    </collision>
-    <inertial>
-      <mass value="0.2"/>
-      <inertia
-        ixx="0.0001" ixy="0.0" ixz="0.0"
-        iyy="0.0001" iyz="0.0"
-        izz="0.0001"/>
-    </inertial>
-  </link>
-  <!-- Joint connecting LIDAR to the robot -->
-  <joint name="laser_frame_joint" type="fixed">
-    <parent link="${parent_link}"/>
-    <child link="laser_frame"/>
-    <origin xyz="0.0 0.0 0.1" rpy="0 0 0"/>
-  </joint>
-</xacro:macro>
+<robot xmlns:xacro="http://ros.org/wiki/xacro">
+  <!-- Xacro file for XV11 LIDAR -->
+  <xacro:macro name="xv11_lidar" parent_link="">
+    <!-- XV11 LIDAR link -->
+    <link name="laser_frame">
+      <visual>
+        <geometry>
+          <!-- Use a cylinder to represent the LIDAR -->
+          <cylinder radius="0.035" length="0.02"/>
+        </geometry>
+        <material name="grey">
+          <color rgba="0.5 0.5 0.5 1.0"/>
+        </material>
+      </visual>
+      <collision>
+        <geometry>
+          <cylinder radius="0.035" length="0.02"/>
+        </geometry>
+      </collision>
+      <inertial>
+        <mass value="0.2"/>
+        <inertia
+          ixx="0.0001" ixy="0.0" ixz="0.0"
+          iyy="0.0001" iyz="0.0"
+          izz="0.0001"/>
+      </inertial>
+    </link>
+    <!-- Joint connecting LIDAR to the robot -->
+    <joint name="laser_frame_joint" type="fixed">
+      <parent link="${parent_link}"/>
+      <child link="laser_frame"/>
+      <origin xyz="0.0 0.0 0.1" rpy="0 0 0"/>
+    </joint>
+  </xacro:macro>
+</robot>

Commit message: Fix bad xacro file for xv11_lidar, take 3

File: turtlebot2_description/urdf/xv11_lidar.urdf.xacro (robot description, xacro)
@@ -2,5 +2,5 @@
 <robot xmlns:xacro="http://ros.org/wiki/xacro">
   <!-- Xacro file for XV11 LIDAR -->
-  <xacro:macro name="xv11_lidar" parent_link="">
+  <xacro:macro name="xv11_lidar" params="parent">
     <!-- XV11 LIDAR link -->
     <link name="laser_frame">
@@ -29,5 +29,5 @@
     <!-- Joint connecting LIDAR to the robot -->
     <joint name="laser_frame_joint" type="fixed">
-      <parent link="${parent_link}"/>
+      <parent link="${parent}"/>
       <child link="laser_frame"/>
       <origin xyz="0.0 0.0 0.1" rpy="0 0 0"/>
